File: hellen-112-17.kicad_pcb (KiCad board)
At the start: 4 copper layers, 86.3 x 97.1 mm, 22 parts, among them J1 rusefi_2x56_pin_conn

Commit message: rev-d
Parts:
- added M1: Module:mega-mcu100-f7/0.2, 0.2:mega-mcu100-f7, F.Cu at (121.4, 138.4)
Routing:
- net (no net): track 147.3 -> 362.4 mm, vias 9 -> 22
- net /IN_DIGITAL_135_HS: track 18.2 -> 93.6 mm
- net +5VA: track 55.9 -> 0.00 mm, vias 5 -> 0
- net /IN_DIGITAL_134_HS: track 24.3 -> 69.3 mm
- net /VREF2: track 29.9 -> 0.00 mm, vias 2 -> 0
- net /DIGITAL_123: track 28.7 -> 0.00 mm, vias 1 -> 0
- net /TLS115_PG: track 26.5 -> 0.00 mm, vias 1 -> 0
- net /DIGITAL_147_HS: track 24.9 -> 0.00 mm, vias 1 -> 0
- net /DIGITAL_136_HS: track 22.0 -> 0.00 mm, vias 1 -> 0
- net /DIGITAL_135_HS: track 14.2 -> 0.00 mm, vias 1 -> 0
- net /DIGITAL_134_HS: track 13.1 -> 0.00 mm, vias 1 -> 0
