File: hellen-112-17.kicad_sch (KiCad schematic)
At the start: 22 parts, among them J1 rusefi_2x56_pin_conn

Commit message: rev-d
Parts:
- added M1: Module:mega-mcu100-f7/0.2, 0.2:mega-mcu100-f7, symbol mega-mcu100-f7:Module{colon}mega-mcu100-f7/0.2
